File: pcb source/zamonaryboard.kicad_pcb (KiCad board)
At the start: 2 copper layers, 52.3 x 40.6 mm, 26 parts, among them J1 USB_C_Receptacle_USB2.0_14P, SW1 SW_Push, U1 ESP32-S2, U2 ME6211C33M5, Y1 Crystal_GND24

Commit message: firmware improvements
Parts:
- removed R6, R7, R8: 0, Resistor_SMD:R_0603_1608Metric
- moved REF** 15.3 mm to (179.3, 95.4)
- moved REF** 15.3 mm to (179.9, 104.8)
- moved R3 1.62 mm to (148.3, 76.0), turned to -90 degrees
- moved C9 0.95 mm to (151.1, 76.3)
- moved R4 0.36 mm to (137.5, 78.3)
Connections:
- C9 pad 2: Net-(C9-Pad2) -> Net-(U1-XTAL_P)
- U1 pad 10: Net-(U1-GPIO5/ADC1_CH4) -> BTN2
- U1 pad 8: Net-(U1-GPIO3/ADC1_CH2) -> BTN1
- Y1 pad 3: Net-(C9-Pad2) -> Net-(U1-XTAL_P)
Routing:
- net BTN2: track 1137.3 -> 1141.9 mm
- net Net-(C9-Pad2): track 3.87 -> 0.00 mm
- net Net-(U1-XTAL_P): track 2.61 -> 6.40 mm
- net Net-(U1-GPIO5/ADC1_CH4): track 3.67 -> 0.00 mm
- net BTN1: track 1121.5 -> 1125.0 mm
- net GND: track 113.2 -> 116.5 mm
- net Net-(U1-GPIO3/ADC1_CH2): track 3.05 -> 0.00 mm
- net Net-(U1-CHIP_PU/RESET): track 17.5 -> 16.7 mm
Other:
- board text added: "since 25.05.2024"
- board text added: "v1"
- board text removed: "0R"
- board text removed: "100nF"
- board text removed: "100pF"
- board text removed: "10K"
- board text removed: "10uF"
- board text removed: "15pF"
- board text removed: "1uF"
- board text removed: "25.05.2024"
- board text removed: "40mHz"
- board text removed: "5.1K"
- board text removed: "500R"
- board text removed: "S2RC"
- board text removed: "prototype 1.4"

Commit message: Python desktop app improvements, PCB pre-v1
Parts:
- removed the REF** at (179.3, 95.4)
- moved REF** 15.3 mm to (164.6, 104.7)
Routing:
- net BTN2: track 1141.9 -> 1115.2 mm
- net BTN1: track 1125.0 -> 1121.1 mm
- net +3V3: track 66.0 -> 66.8 mm
Other:
- board text added: "40.64mm"
- board text added: "52.32mm"
- board text removed: "40.640mm"
- board text removed: "52.324mm"
- board text removed: "GND"
- board text removed: "This work is licensed under CC BY-SA 4.0. To view a copy of this license, visit https://creativecommons.org/licenses/by-sa/4.0/"

Commit message: v1 commit, desktop app improvements
Parts:
- removed C5: 100nF, Capacitor_SMD:C_0603_1608Metric
- moved C4 1.63 mm to (123.3, 82.0)
- moved C9 0.20 mm to (151.1, 76.5)
Routing:
- net BTN2: track 1115.2 -> 1137.9 mm
- net BTN1: track 1121.1 -> 1142.9 mm
- net +3V3: track 66.8 -> 64.5 mm
- net GND: track 116.5 -> 114.7 mm
Other:
- board text removed: "since 25.05.2024"
